Commit message: correct cameras position

File: urdf/koala.xacro (robot description, xacro)
@@ -44,9 +44,16 @@
   <xacro:sensor_d435 parent="depth_link" use_nominal_extrinsics="true" add_plug="false" use_mesh="true">
       <origin xyz="0 0 0" rpy="0 0 0"/>
-    </xacro:sensor_d435>
+  </xacro:sensor_d435>
+  <link name="stereo_link">
+  </link>
   <joint name="frame_to_depth" type="fixed" >
-    <origin xyz="0.08 0.0 -0.13" rpy="0.0 0.95 0.0" />
+    <origin xyz="0.1085 0.0 -0.0734" rpy="0.0 1.221 0.0" />
     <parent link="drone_frame" />
     <child link="depth_link" />
+  </joint>
+  <joint name="frame_to_stereo" type="fixed" >
+    <origin xyz="-0.485 0.0 -0.08" rpy="0.0 0.0 3.14" />
+    <parent link="drone_frame" />
+    <child link="stereo_link" />
   </joint>
   <joint name="base_to_frame" type="fixed" >

Commit message: added application launch file

File: urdf/koala.xacro (robot description, xacro)
@@ -1,5 +1,8 @@
 <?xml version="1.0" ?>
 <robot name="koala" xmlns:xacro="http://www.ros.org/wiki/xacro">
-  <xacro:include filename="$(find realsense2_description)/urdf/_d435.urdf.xacro" />
+  <xacro:arg name="is_simulation" default="true" />
+  <xacro:if value="$(arg is_simulation)">
+    <xacro:include filename="$(find realsense2_description)/urdf/_d435.urdf.xacro" />
+  </xacro:if>
   <material name="silver">
     <color rgba="0.700 0.700 0.700 1.000"/>
@@ -40,20 +43,22 @@
     </visual>
   </link>
-  <link name="depth_link">
+  <link name="d400_link">
   </link>
-  <xacro:sensor_d435 parent="depth_link" use_nominal_extrinsics="true" add_plug="false" use_mesh="true">
-      <origin xyz="0 0 0" rpy="0 0 0"/>
-  </xacro:sensor_d435>
-  <link name="stereo_link">
+  <xacro:if value="$(arg is_simulation)">
+    <xacro:sensor_d435 parent="d400_link" use_nominal_extrinsics="true" add_plug="false" use_mesh="true">
+        <origin xyz="0 0 0" rpy="0 0 0"/>
+    </xacro:sensor_d435>
+  </xacro:if>
+  <link name="t265_link">
   </link>
   <joint name="frame_to_depth" type="fixed" >
     <origin xyz="0.1085 0.0 -0.0734" rpy="0.0 1.221 0.0" />
     <parent link="drone_frame" />
-    <child link="depth_link" />
+    <child link="d400_link" />
   </joint>
   <joint name="frame_to_stereo" type="fixed" >
     <origin xyz="-0.485 0.0 -0.08" rpy="0.0 0.0 3.14" />
     <parent link="drone_frame" />
-    <child link="stereo_link" />
+    <child link="t265_link" />
   </joint>
   <joint name="base_to_frame" type="fixed" >

Commit message: simulation working with upside and downside config

File: urdf/koala.xacro (robot description, xacro)
@@ -2,7 +2,7 @@
 <robot name="koala" xmlns:xacro="http://www.ros.org/wiki/xacro">
   <xacro:arg name="is_simulation" default="true" />
-  <xacro:if value="$(arg is_simulation)">
+  <!-- <xacro:if value="$(arg is_simulation)">
     <xacro:include filename="$(find realsense2_description)/urdf/_d435.urdf.xacro" />
-  </xacro:if>
+  </xacro:if> -->
   <material name="silver">
     <color rgba="0.700 0.700 0.700 1.000"/>
@@ -43,23 +43,23 @@
     </visual>
   </link>
-  <link name="d400_link">
-  </link>
-  <xacro:if value="$(arg is_simulation)">
-    <xacro:sensor_d435 parent="d400_link" use_nominal_extrinsics="true" add_plug="false" use_mesh="true">
+  <!-- <link name="d400_link">
+  </link> -->
+  <!-- <xacro:if value="$(arg is_simulation)">
+    <xacro:sensor_d435 parent="pipecam_link" use_nominal_extrinsics="true" add_plug="false" use_mesh="true">
         <origin xyz="0 0 0" rpy="0 0 0"/>
     </xacro:sensor_d435>
-  </xacro:if>
-  <link name="t265_link">
-  </link>
-  <joint name="frame_to_depth" type="fixed" >
+  </xacro:if> -->
+  <!-- <link name="t265_link">
+  </link> -->
+  <!-- <joint name="frame_to_depth" type="fixed" >
     <origin xyz="0.1085 0.0 -0.0734" rpy="0.0 1.221 0.0" />
     <parent link="drone_frame" />
     <child link="d400_link" />
-  </joint>
-  <joint name="frame_to_stereo" type="fixed" >
+  </joint> -->
+  <!-- <joint name="frame_to_stereo" type="fixed" >
     <origin xyz="-0.485 0.0 -0.08" rpy="0.0 0.0 3.14" />
     <parent link="drone_frame" />
     <child link="t265_link" />
-  </joint>
+  </joint> -->
   <joint name="base_to_frame" type="fixed" >
     <origin xyz="0.0 0.0 0.0" rpy="0.0 0.0 0.0" />
